Commit message: Moved files from test to demo directory

File: demo/demo.xacro (robot description, xacro)
@@ -6,5 +6,5 @@
     <visual>
       <geometry>
-        <mesh filename="package://simulated_lidar_scanner/test/view_object.stl"/>
+        <mesh filename="package://simulated_lidar_scanner/demo/view_object.stl"/>
       </geometry>
       <material name="view_object_material">
